Commit message: Added SLAM Toolbox

File: src/sim/urdf/robot.urdf.xacro (robot description, xacro)
@@ -2,4 +2,5 @@
 <robot xmlns:xacro="http://www.ros.org/wiki/xacro" name="my_robot">
     <xacro:include filename="ros2_control.xacro" />
+    <xacro:include filename="lidar.xacro" />
     <!-- BASE LINK (free floating) -->
     <link name="base_link"></link>
@@ -10,4 +11,12 @@
         <origin xyz="0 0 0" rpy="0 0 0"/>
     </joint>
+    <!-- BASE_FOOTPRINT LINK -->
+    <joint name="base_footprint_joint" type="fixed">
+        <parent link="base_link"/>
+        <child link="base_footprint"/>
+        <origin xyz="0 0 0" rpy="0 0 0"/>
+    </joint>
+    <link name="base_footprint">
+    </link>
     <link name="body_link">
     <visual>
